Commit message: Agregar pika_sim: Piper + gripper Pika simulado en Gazebo para teleop sin hardware
Paquete nuevo src/pika_sim (Flujo D+):
- piper_sim_bridge.py: reemplaza al driver CAN con su mismo contrato de topics
  (/joint_states_gripper -> Gazebo -> /joint_states_single, 200 Hz). Reordena
  por nombre el estado de Gazebo, porque FK/IK leen position[:6].
- fake_pika_sense.py: marcador interactivo en RViz como Pika Sense + Vive
  (/pika_pose, mezcla de apertura en /joint_states_gripper, /teleop_trigger).
- sim_piper_single.launch.py (sense:=fake|real, gui, rviz), URDF con
  ros2_control, controladores de posicion, config de RViz.

Probado headless contra los nodos reales de teleop (conda pika): arrastrar el
marcador 5 cm mueve el TCP ~4.8 cm en el marco de la herramienta.

pika_description: pika_piper_standalone no parseaba con el piper_description
de este workspace (raiz dummy_link -> dos raices). Nuevo argumento arm_root
(default dummy_link; base_link para ~/piper_ros), tambien en
display_pika_piper.launch.py.

Submodulo PikaAnyArm: argumento sim:=true en teleop_rand_single_piper.launch.py.

Co-Authored-By: Claude Opus 5.5 <noreply@anthropic.com>

File: src/pika_description/urdf/pika_piper_standalone.urdf.xacro (robot description, xacro)
@@ -13,5 +13,9 @@
 <robot name="pika_piper" xmlns:xacro="http://ros.org/wiki/xacro">
   <xacro:arg name="gripper" default="pika"/>
-  <!-- Piper arm (base_link es root en el .urdf original, sin world) -->
+  <!-- Link raíz del URDF del Piper: el piper_description de este workspace
+       (src/PikaAnyArm) empieza en dummy_link; el de ~/piper_ros empieza en
+       base_link (usar arm_root:=base_link si es ese el que queda en el path) -->
+  <xacro:arg name="arm_root" default="dummy_link"/>
+  <!-- Piper arm -->
   <xacro:include filename="$(find piper_description)/urdf/piper_no_gripper_description.urdf"/>
   <!-- Frame raíz explícito -->
@@ -19,5 +23,5 @@
   <joint name="world_to_base" type="fixed">
     <parent link="world"/>
-    <child link="base_link"/>
+    <child link="$(arg arm_root)"/>
     <origin xyz="0 0 0" rpy="0 0 0"/>
   </joint>
