Commit message: add interchangeable gripper support to pika_piper URDF
- pika_piper_standalone.urdf.xacro: add xacro:arg 'gripper' (default: pika)
  with xacro:if blocks per gripper type and placeholder for future grippers
- display_pika_piper.launch.py: add 'gripper' launch argument resolved via
  OpaqueFunction so xacro mappings are applied at launch time
- add world link + world_to_base fixed joint so TF tree is rooted at 'world'
- add rviz/pika_piper.rviz config for the full arm visualization

Co-Authored-By: Claude Sonnet 4.6 <noreply@anthropic.com>

File: src/pika_description/urdf/pika_gripper_macro.urdf.xacro (robot description, xacro)
@@ -57,48 +57,4 @@
         <mass value="0.450"/>
         <inertia ixx="9.3e-4" ixy="3.4e-7" ixz="-7.4e-6" iyy="7.1e-4" iyz="5e-8" izz="3.9e-4"/>
-      </inertial>
-    </link>
-    <!-- ══════════════════════════════════════════════════════════════
-         DEPTH CAMERA — Intel RealSense D405
-         46 mm sobre el eje del gripper → Z = 0.1358 - 0.046 = 0.0898 m
-    ══════════════════════════════════════════════════════════════════ -->
-    <joint name="${prefix}pika_depth_joint" type="fixed">
-      <parent link="${prefix}gripper_base"/>
-      <child  link="${prefix}pika_depth_link"/>
-      <origin xyz="0 0.095 0.0898" rpy="0 0 0"/>
-    </joint>
-    <link name="${prefix}pika_depth_link">
-      <visual>
-        <origin xyz="0 0 0" rpy="0 0 0"/>
-        <geometry>
-          <mesh filename="package://realsense2_description/meshes/d405.stl"
-                scale="0.001 0.001 0.001"/>
-        </geometry>
-        <material name="${prefix}pika_aluminum"/>
-      </visual>
-      <collision>
-        <origin xyz="0 -0.0115 0" rpy="0 0 0"/>
-        <geometry><box size="0.042 0.023 0.042"/></geometry>
-      </collision>
-      <inertial>
-        <mass value="0.072"/>
-        <inertia ixx="3.88e-6" ixy="0" ixz="0" iyy="4.99e-7" iyz="0" izz="3.88e-6"/>
-      </inertial>
-    </link>
-    <!-- ══════════════════════════════════════════════════════════════
-         FISHEYE CAMERA (广角单目, FOV diagonal 200°)
-         73.5 mm sobre el eje del gripper → Z = 0.1358 - 0.0735 = 0.0623 m
-         TODO: reemplazar por malla real
-    ══════════════════════════════════════════════════════════════════ -->
-    <joint name="${prefix}pika_fisheye_joint" type="fixed">
-      <parent link="${prefix}gripper_base"/>
-      <child  link="${prefix}pika_fisheye_link"/>
-      <!-- rpy="-1.5708 0 0": child +Z apunta a pika +Y (hacia workspace) -->
-      <origin xyz="0 0.092 0.0623" rpy="-1.5708 0 0"/>
-    </joint>
-    <link name="${prefix}pika_fisheye_link">
-      <inertial>
-        <mass value="0.008"/>
-        <inertia ixx="1e-6" ixy="0" ixz="0" iyy="1e-6" iyz="0" izz="1e-6"/>
       </inertial>
     </link>

Commit message: restore D405 and fisheye camera links in pika_gripper_macro
Cameras were temporarily removed to isolate jaw oscillation bug.
Root cause was multiple robot_state_publisher instances, not cameras.

Co-Authored-By: Claude Sonnet 4.6 <noreply@anthropic.com>

File: src/pika_description/urdf/pika_gripper_macro.urdf.xacro (robot description, xacro)
@@ -57,4 +57,47 @@
         <mass value="0.450"/>
         <inertia ixx="9.3e-4" ixy="3.4e-7" ixz="-7.4e-6" iyy="7.1e-4" iyz="5e-8" izz="3.9e-4"/>
+      </inertial>
+    </link>
+    <!-- ══════════════════════════════════════════════════════════════
+         DEPTH CAMERA — Intel RealSense D405
+         46 mm sobre el eje del gripper → Z = 0.1358 - 0.046 = 0.0898 m
+    ══════════════════════════════════════════════════════════════════ -->
+    <joint name="${prefix}pika_depth_joint" type="fixed">
+      <parent link="${prefix}gripper_base"/>
+      <child  link="${prefix}pika_depth_link"/>
+      <origin xyz="0 0.095 0.0898" rpy="0 0 0"/>
+    </joint>
+    <link name="${prefix}pika_depth_link">
+      <visual>
+        <origin xyz="0 0 0" rpy="0 0 0"/>
+        <geometry>
+          <mesh filename="package://realsense2_description/meshes/d405.stl"
+                scale="0.001 0.001 0.001"/>
+        </geometry>
+        <material name="${prefix}pika_aluminum"/>
+      </visual>
+      <collision>
+        <origin xyz="0 -0.0115 0" rpy="0 0 0"/>
+        <geometry><box size="0.042 0.023 0.042"/></geometry>
+      </collision>
+      <inertial>
+        <mass value="0.072"/>
+        <inertia ixx="3.88e-6" ixy="0" ixz="0" iyy="4.99e-7" iyz="0" izz="3.88e-6"/>
+      </inertial>
+    </link>
+    <!-- ══════════════════════════════════════════════════════════════
+         FISHEYE CAMERA (广角单目, FOV diagonal 200°)
+         73.5 mm sobre el eje del gripper → Z = 0.1358 - 0.0735 = 0.0623 m
+         TODO: reemplazar por malla real
+    ══════════════════════════════════════════════════════════════════ -->
+    <joint name="${prefix}pika_fisheye_joint" type="fixed">
+      <parent link="${prefix}gripper_base"/>
+      <child  link="${prefix}pika_fisheye_link"/>
+      <origin xyz="0 0.092 0.0623" rpy="-1.5708 0 0"/>
+    </joint>
+    <link name="${prefix}pika_fisheye_link">
+      <inertial>
+        <mass value="0.008"/>
+        <inertia ixx="1e-6" ixy="0" ixz="0" iyy="1e-6" iyz="0" izz="1e-6"/>
       </inertial>
     </link>

Commit message: make pika_description self-contained: copy meshes locally
- add meshes/: gripper_base.STL, link7.STL, link8.STL (from piper_description),
  d405.stl (from realsense2_description)
- update pika_gripper_macro to reference package://pika_description/meshes/
- remove exec_depend on piper_description and realsense2_description
- add meshes/ to CMakeLists install targets

pika_description no longer depends on piper_ros at runtime for mesh files.

Co-Authored-By: Claude Sonnet 4.6 <noreply@anthropic.com>

File: src/pika_description/urdf/pika_gripper_macro.urdf.xacro (robot description, xacro)
@@ -44,5 +44,5 @@
         <origin xyz="0 0 0" rpy="0 0 0"/>
         <geometry>
-          <mesh filename="package://piper_description/meshes/gripper_base.STL"/>
+          <mesh filename="package://pika_description/meshes/gripper_base.STL"/>
         </geometry>
         <material name="${prefix}pika_mid"/>
@@ -51,5 +51,5 @@
         <origin xyz="0 0 0" rpy="0 0 0"/>
         <geometry>
-          <mesh filename="package://piper_description/meshes/gripper_base.STL"/>
+          <mesh filename="package://pika_description/meshes/gripper_base.STL"/>
         </geometry>
       </collision>
@@ -72,5 +72,5 @@
         <origin xyz="0 0 0" rpy="0 0 0"/>
         <geometry>
-          <mesh filename="package://realsense2_description/meshes/d405.stl"
+          <mesh filename="package://pika_description/meshes/d405.stl"
                 scale="0.001 0.001 0.001"/>
         </geometry>
@@ -117,5 +117,5 @@
         <origin xyz="0 0 0" rpy="0 0 0"/>
         <geometry>
-          <mesh filename="package://piper_description/meshes/link7.STL"/>
+          <mesh filename="package://pika_description/meshes/link7.STL"/>
         </geometry>
         <material name="${prefix}pika_dark"/>
@@ -124,5 +124,5 @@
         <origin xyz="0 0 0" rpy="0 0 0"/>
         <geometry>
-          <mesh filename="package://piper_description/meshes/link7.STL"/>
+          <mesh filename="package://pika_description/meshes/link7.STL"/>
         </geometry>
       </collision>
@@ -144,5 +144,5 @@
         <origin xyz="0 0 0" rpy="0 0 0"/>
         <geometry>
-          <mesh filename="package://piper_description/meshes/link8.STL"/>
+          <mesh filename="package://pika_description/meshes/link8.STL"/>
         </geometry>
         <material name="${prefix}pika_dark"/>
@@ -151,5 +151,5 @@
         <origin xyz="0 0 0" rpy="0 0 0"/>
         <geometry>
-          <mesh filename="package://piper_description/meshes/link8.STL"/>
+          <mesh filename="package://pika_description/meshes/link8.STL"/>
         </geometry>
       </collision>

Commit message: update D405 camera position and orientation from technical drawings
- Position from Agilex datasheet: X=-0.132m, Z=0.0908m (45mm above jaw axis)
- Fisheye position updated: Y=0.122m (122mm from flange per drawing)
- D405 visual rpy="0 3.1416 1.5708" (90° Z + 180° Y) for correct mesh orientation

Co-Authored-By: Claude Sonnet 4.6 <noreply@anthropic.com>

File: src/pika_description/urdf/pika_gripper_macro.urdf.xacro (robot description, xacro)
@@ -4,9 +4,9 @@
   Paquete autónomo — todas las mallas están en pika_description/meshes/.
   No requiere piper_ros ni realsense2_description en tiempo de ejecución.
-  Dimensiones de referencia:
+  Dimensiones de referencia (plano técnico Agilex):
     Eje de garras:  0.1358 m desde gripper_base (igual que joint7/joint8 del Piper)
     Apertura máx:   ±35 mm por lado
-    Cámara D405:    centrada en X, 46 mm sobre el eje del gripper  → Z = 0.0898 m
-    Fisheye (广角): centrada en X, 73.5 mm sobre el eje del gripper → Z = 0.0623 m
+    Cámara D405:    X=0, Y=132 mm desde brida, Z=90.8 mm (45 mm sobre eje garras)
+    Fisheye (广角): X=0, Y=122 mm desde brida, Z=62.3 mm (73.5 mm sobre eje garras)
   Marco de coordenadas (gripper_base):
     Origen = cara de la brida (interfaz con link6 / parent)
@@ -62,14 +62,15 @@
     <!-- ══════════════════════════════════════════════════════════════
          DEPTH CAMERA — Intel RealSense D405
-         46 mm sobre el eje del gripper → Z = 0.1358 - 0.046 = 0.0898 m
+         Plano técnico: 132 mm desde brida (Y), 45 mm sobre eje garras (Z)
+         Z = 0.1358 - 0.045 = 0.0908 m
     ══════════════════════════════════════════════════════════════════ -->
     <joint name="${prefix}pika_depth_joint" type="fixed">
       <parent link="${prefix}gripper_base"/>
       <child  link="${prefix}pika_depth_link"/>
-      <origin xyz="0 0.095 0.0898" rpy="0 0 0"/>
+      <origin xyz="-0.132 0 0.0908" rpy="0 0 0"/>
     </joint>
     <link name="${prefix}pika_depth_link">
       <visual>
-        <origin xyz="0 0 0" rpy="0 0 0"/>
+        <origin xyz="0 0 0" rpy="0 3.1416 1.5708"/>
         <geometry>
           <mesh filename="package://pika_description/meshes/d405.stl"
@@ -79,5 +80,5 @@
       </visual>
       <collision>
-        <origin xyz="0 -0.0115 0" rpy="0 0 0"/>
+        <origin xyz="0 -0.0115 0" rpy="0 3.1416 1.5708"/>
         <geometry><box size="0.042 0.023 0.042"/></geometry>
       </collision>
@@ -89,5 +90,6 @@
     <!-- ══════════════════════════════════════════════════════════════
          FISHEYE CAMERA (广角单目, FOV diagonal 200°)
-         73.5 mm sobre el eje del gripper → Z = 0.1358 - 0.0735 = 0.0623 m
+         Plano técnico: 122 mm desde brida (Y), 73.5 mm sobre eje garras (Z)
+         Z = 0.1358 - 0.0735 = 0.0623 m
          TODO: reemplazar por malla real
     ══════════════════════════════════════════════════════════════════ -->
@@ -95,5 +97,5 @@
       <parent link="${prefix}gripper_base"/>
       <child  link="${prefix}pika_fisheye_link"/>
-      <origin xyz="0 0.092 0.0623" rpy="-1.5708 0 0"/>
+      <origin xyz="0 0.122 0.0623" rpy="-1.5708 0 0"/>
     </joint>
     <link name="${prefix}pika_fisheye_link">

Commit message: pika_description: posición/orientación final de cámaras D405 y fisheye
- Añade malla fisheye.stl (WN-L712V11) al pika_fisheye_link, antes sin visual
- Ajusta posición de cámaras sobre gripper_base (D405 -0.046/0/0.027,
  fisheye -0.0735/0/0.037) y orientación de visuals
- Actualiza README y comentarios del xacro con valores reales
- Manual.md: añade flujo de pipeline de datos y config CAN dual (can_config.sh)
- Bump punteros submódulos data_msgs, data_tools, PikaAnyArm (can paths del host)

Co-Authored-By: Claude Opus 4.8 <noreply@anthropic.com>

File: src/pika_description/urdf/pika_gripper_macro.urdf.xacro (robot description, xacro)
@@ -7,6 +7,6 @@
     Eje de garras:  0.1358 m desde gripper_base (igual que joint7/joint8 del Piper)
     Apertura máx:   ±35 mm por lado
-    Cámara D405:    X=0, Y=132 mm desde brida, Z=90.8 mm (45 mm sobre eje garras)
-    Fisheye (广角): X=0, Y=122 mm desde brida, Z=62.3 mm (73.5 mm sobre eje garras)
+    Cámara D405:    X=-46 mm (largo del gripper), Z=27 mm (altura), Y=0
+    Fisheye (广角): X=-73.5 mm (largo del gripper), Z=37 mm (altura), Y=0
   Marco de coordenadas (gripper_base):
     Origen = cara de la brida (interfaz con link6 / parent)
@@ -19,6 +19,5 @@
     - pika_jaw_right    : link8.STL
     - pika_depth_link   : d405.stl
-  Visuals pendientes:
-    - pika_fisheye_link : TODO malla real
+    - pika_fisheye_link : fisheye.stl (WN-L712V11)
 -->
 <robot xmlns:xacro="http://ros.org/wiki/xacro">
@@ -62,11 +61,11 @@
     <!-- ══════════════════════════════════════════════════════════════
          DEPTH CAMERA — Intel RealSense D405
-         Plano técnico: 132 mm desde brida (Y), 45 mm sobre eje garras (Z)
-         Z = 0.1358 - 0.045 = 0.0908 m
+         Posición sobre gripper_base: X=-46 mm (a lo largo del gripper),
+         Z=27 mm (altura). Y=0.
     ══════════════════════════════════════════════════════════════════ -->
     <joint name="${prefix}pika_depth_joint" type="fixed">
       <parent link="${prefix}gripper_base"/>
       <child  link="${prefix}pika_depth_link"/>
-      <origin xyz="-0.132 0 0.0908" rpy="0 0 0"/>
+      <origin xyz="-0.046 0 0.027" rpy="0 0 0"/>
     </joint>
     <link name="${prefix}pika_depth_link">
@@ -89,15 +88,27 @@
     </link>
     <!-- ══════════════════════════════════════════════════════════════
-         FISHEYE CAMERA (广角单目, FOV diagonal 200°)
-         Plano técnico: 122 mm desde brida (Y), 73.5 mm sobre eje garras (Z)
-         Z = 0.1358 - 0.0735 = 0.0623 m
-         TODO: reemplazar por malla real
+         FISHEYE CAMERA (广角单目, FOV diagonal 200°) — WN-L712V11
+         Posición sobre gripper_base: X=-73.5 mm (a lo largo del gripper),
+         Z=37 mm (altura). Y=0.
+         Malla: fisheye.stl (Ø22.65 × 20.2 mm, exportada de SolidWorks→Onshape)
     ══════════════════════════════════════════════════════════════════ -->
     <joint name="${prefix}pika_fisheye_joint" type="fixed">
       <parent link="${prefix}gripper_base"/>
       <child  link="${prefix}pika_fisheye_link"/>
-      <origin xyz="0 0.122 0.0623" rpy="-1.5708 0 0"/>
+      <origin xyz="-0.0735 0 0.037" rpy="-1.5708 0 0"/>
     </joint>
     <link name="${prefix}pika_fisheye_link">
+      <visual>
+        <origin xyz="0 0 0" rpy="1.5708 0 0"/>
+        <geometry>
+          <mesh filename="package://pika_description/meshes/fisheye.stl"
+                scale="0.001 0.001 0.001"/>
+        </geometry>
+        <material name="${prefix}pika_dark"/>
+      </visual>
+      <collision>
+        <origin xyz="0 0 0.0045" rpy="1.5708 0 0"/>
+        <geometry><cylinder radius="0.0113" length="0.0202"/></geometry>
+      </collision>
       <inertial>
         <mass value="0.008"/>
