Commit message: Modelo oficial de AgileX del gripper Pika y del Sense
- pika_description: mallas y medidas de pika_gripper_description (AgileX),
  pasadas al marco del link6 del Piper; mismos nombres de links y joints.
  Garras a lo largo de Y, apertura 0-94 mm; D405 y fisheye en las posiciones
  del plano de AgileX, mirando por el eje de la herramienta; TCP a 0,180 m.
  Masa de la base escalada al peso publicado (617 g); colisiones con cajas.
- agilex/: URDF, CSV y planos originales, con su procedencia. Los STEP no
  se guardan en el repo.
- pika_sim: camaras del gripper en los marcos nuevos (D405 4 mm delante de
  la tapa); apertura 0-94 mm en el puente, el Sense falso y la demo; el Sense
  falso usa la malla del Pika Sense de AgileX.
- T_FF del modo MIT recalculado con el gripper nuevo (sigue estable).
- Figuras de PIPER_PIKA.md regeneradas; documentacion actualizada (TCP,
  apertura, frutas que caben, camaras confirmadas).

Archivos de AgileX entregados en privado: no publicar sin su permiso.

Co-Authored-By: Claude Opus 5.5 <noreply@anthropic.com>

File: src/pika_description/urdf/pika_gripper_macro.urdf.xacro (robot description, xacro)
@@ -1,37 +1,38 @@
 <?xml version="1.0"?>
 <!--
-  Pika Gripper URDF — Agilex Robotics
-  Paquete autónomo — todas las mallas están en pika_description/meshes/.
-  No requiere piper_ros ni realsense2_description en tiempo de ejecución.
-  Dimensiones de referencia (plano técnico Agilex):
-    Eje de garras:  0.1358 m desde gripper_base (igual que joint7/joint8 del Piper)
-    Apertura máx:   ±35 mm por lado
-    Cámara D405:    X=-46 mm (largo del gripper), Z=27 mm (altura), Y=0
-    Fisheye (广角): X=-73.5 mm (largo del gripper), Z=37 mm (altura), Y=0
-  Marco de coordenadas (gripper_base):
-    Origen = cara de la brida (interfaz con link6 / parent)
-    +Z  : hacia las garras (eje herramienta)
-    +X  : apertura de las garras
-    +Y  : cara frontal (hacia el espacio de trabajo)
-  Visuals activos (meshes en pika_description/meshes/):
-    - gripper_base      : gripper_base.STL
-    - pika_jaw_left     : link7.STL
-    - pika_jaw_right    : link8.STL
-    - pika_depth_link   : d405.stl
-    - pika_fisheye_link : fisheye.stl (WN-L712V11)
+  Pika Gripper URDF — modelo oficial de AgileX Robotics
+  Mallas y medidas de pika_gripper_description, enviado por el soporte de AgileX el 20-10-2026
+  (originales en pika_description/agilex/). Este macro los pasa al marco de este repositorio y
+  conserva los nombres de links y joints que usan pika_sim y la teleop.
+  Marco de coordenadas (gripper_base), el mismo que el link6 del Piper:
+    Origen = cara de la brida (interfaz con link6)
+    +Z : eje de la herramienta, hacia las puntas de las garras
+    +Y : dirección en que se desplazan las garras
+    −X : lado de las cámaras
+  AgileX usa otro marco (X herramienta, Y garras, Z cámaras): el paso es
+    x = −z_AgileX,  y = y_AgileX,  z = x_AgileX   (rpy 0 −π/2 0 en las mallas)
+  Medidas (mallas de AgileX y plano de cámaras):
+    Puntas de las garras:  z = 0,190 m desde la brida (el plano da 194,3 mm desde la base del montaje)
+    Apertura:              0 a 94 mm entre las caras internas (cada garra 0 a 47 mm); el driver real
+                           limita la apertura total a 98 mm
+    Cámara D405:           46 mm sobre el eje de las garras, cara a 132 mm de las puntas; el marco va en
+                           el imager izquierdo (línea base de 18 mm)
+    Fisheye:               73,5 mm sobre el eje de las garras, lente a 122 mm de las puntas
+    Ambas cámaras miran a lo largo de +Z (eje de la herramienta), según el plano de AgileX.
+    TCP (pika_tcp):        entre las garras, a 0,180 m (1 cm detrás de las puntas)
+  Masa: las inercias del CAD de AgileX suman 0,257 kg, pero el gripper pesa 617–690 g según las
+  tiendas (con motor y cámaras). La base se escala a 0,55 kg (total 0,617 kg), con el centro de masa
+  y la forma de la inercia del CAD.
 -->
 <robot xmlns:xacro="http://ros.org/wiki/xacro">
   <xacro:macro name="pika_gripper" params="prefix:='' parent origin_xyz:='0 0 0' origin_rpy:='0 0 0'">
-    <!-- ── Materiales ────────────────────────────────────────────────── -->
+    <xacro:property name="AGILEX" value="0 -1.5708 0"/>   <!-- rotación de las mallas de AgileX -->
+    <xacro:property name="MALLAS" value="package://pika_description/meshes/agilex/gripper"/>
+    <material name="${prefix}pika_dark">
+      <color rgba="0.18 0.18 0.18 1.0"/>
+    </material>
     <material name="${prefix}pika_mid">
       <color rgba="0.55 0.55 0.55 1.0"/>
     </material>
-    <material name="${prefix}pika_dark">
-      <color rgba="0.18 0.18 0.18 1.0"/>
-    </material>
-    <material name="${prefix}pika_aluminum">
-      <color rgba="0.75 0.75 0.80 1.0"/>
-    </material>
-    <!-- ── Junta de montaje → gripper_base (= joint6_to_gripper_base del Piper) ── -->
     <joint name="${prefix}pika_mount_joint" type="fixed">
       <parent link="${parent}"/>
@@ -39,143 +40,91 @@
       <origin xyz="${origin_xyz}" rpy="${origin_rpy}"/>
     </joint>
-    <!-- gripper_base — mismo STL que el Piper -->
+    <!-- Cuerpo: carcasa, motor, D405 y fisheye (todo en una malla) -->
     <link name="${prefix}gripper_base">
       <visual>
-        <origin xyz="0 0 0" rpy="0 0 0"/>
-        <geometry>
-          <mesh filename="package://pika_description/meshes/gripper_base.STL"/>
-        </geometry>
+        <origin xyz="0 0 0" rpy="${AGILEX}"/>
+        <geometry><mesh filename="${MALLAS}/gripper_base_link.STL"/></geometry>
+        <material name="${prefix}pika_dark"/>
+      </visual>
+      <collision>
+        <origin xyz="-0.0335 0 0.0424" rpy="0 0 0"/>
+        <geometry><box size="0.143 0.215 0.0848"/></geometry>
+      </collision>
+      <inertial>
+        <origin xyz="-0.00841 0 0.03748" rpy="0 0 0"/>
+        <mass value="0.55"/>
+        <inertia ixx="0.00032" ixy="-4.9e-08" ixz="7.6e-06" iyy="0.000415" iyz="9.7e-08" izz="0.000626"/>
+      </inertial>
+    </link>
+    <!-- Garras: prismáticas a lo largo de Y. El origen del joint es la garra cerrada; q es la mitad
+         de la apertura (caras internas a 2q), como el driver real reparte la apertura total. -->
+    <joint name="${prefix}pika_jaw_left_joint" type="prismatic">
+      <parent link="${prefix}gripper_base"/>
+      <child  link="${prefix}pika_jaw_left"/>
+      <origin xyz="-0.00642 0.0415 0.0815" rpy="0 0 0"/>
+      <axis xyz="0 1 0"/>
+      <limit lower="0" upper="0.047" effort="10.0" velocity="1.0"/>
+    </joint>
+    <link name="${prefix}pika_jaw_left">
+      <visual>
+        <origin xyz="0 0 0" rpy="${AGILEX}"/>
+        <geometry><mesh filename="${MALLAS}/gripper_left_link.STL"/></geometry>
         <material name="${prefix}pika_mid"/>
       </visual>
       <collision>
-        <origin xyz="0 0 0" rpy="0 0 0"/>
-        <geometry>
-          <mesh filename="package://pika_description/meshes/gripper_base.STL"/>
-        </geometry>
+        <origin xyz="0.00575 -0.013 0.05275" rpy="0 0 0"/>
+        <geometry><box size="0.0381 0.057 0.1121"/></geometry>
       </collision>
       <inertial>
-        <mass value="0.450"/>
-        <inertia ixx="9.3e-4" ixy="3.4e-7" ixz="-7.4e-6" iyy="7.1e-4" iyz="5e-8" izz="3.9e-4"/>
+        <origin xyz="0.00576 -0.01466 0.03326" rpy="0 0 0"/>
+        <mass value="0.0337"/>
+        <inertia ixx="3.974e-05" ixy="4.4e-09" ixz="-1.5e-08" iyy="3.448e-05" iyz="1.447e-05" izz="1.528e-05"/>
       </inertial>
     </link>
-    <!-- ══════════════════════════════════════════════════════════════
-         DEPTH CAMERA — Intel RealSense D405
-         Posición sobre gripper_base: X=-46 mm (a lo largo del gripper),
-         Z=27 mm (altura). Y=0.
-    ══════════════════════════════════════════════════════════════════ -->
+    <joint name="${prefix}pika_jaw_right_joint" type="prismatic">
+      <parent link="${prefix}gripper_base"/>
+      <child  link="${prefix}pika_jaw_right"/>
+      <origin xyz="-0.00642 -0.0415 0.0815" rpy="0 0 0"/>
+      <axis xyz="0 1 0"/>
+      <limit lower="-0.047" upper="0" effort="10.0" velocity="1.0"/>
+    </joint>
+    <link name="${prefix}pika_jaw_right">
+      <visual>
+        <origin xyz="0 0 0" rpy="${AGILEX}"/>
+        <geometry><mesh filename="${MALLAS}/gripper_right_link.STL"/></geometry>
+        <material name="${prefix}pika_mid"/>
+      </visual>
+      <collision>
+        <origin xyz="0.00575 0.013 0.05275" rpy="0 0 0"/>
+        <geometry><box size="0.0381 0.057 0.1121"/></geometry>
+      </collision>
+      <inertial>
+        <origin xyz="0.00581 0.01466 0.03326" rpy="0 0 0"/>
+        <mass value="0.0337"/>
+        <inertia ixx="3.974e-05" ixy="4.4e-09" ixz="1.5e-08" iyy="3.448e-05" iyz="-1.447e-05" izz="1.528e-05"/>
+      </inertial>
+    </link>
+    <!-- Cámaras: solo marcos (la malla está en el cuerpo). Inercia mínima para que Gazebo no los
+         descarte junto con los sensores que cuelgan de ellos. -->
     <joint name="${prefix}pika_depth_joint" type="fixed">
       <parent link="${prefix}gripper_base"/>
       <child  link="${prefix}pika_depth_link"/>
-      <origin xyz="-0.046 0 0.027" rpy="0 0 0"/>
+      <origin xyz="-0.0524 0.009 0.0583" rpy="0 0 0"/>
     </joint>
     <link name="${prefix}pika_depth_link">
-      <visual>
-        <origin xyz="0 0 0" rpy="0 3.1416 1.5708"/>
-        <geometry>
-          <mesh filename="package://pika_description/meshes/d405.stl"
-                scale="0.001 0.001 0.001"/>
-        </geometry>
-        <material name="${prefix}pika_aluminum"/>
-      </visual>
-      <collision>
-        <origin xyz="0 -0.0115 0" rpy="0 3.1416 1.5708"/>
-        <geometry><box size="0.042 0.023 0.042"/></geometry>
-      </collision>
-      <inertial>
-        <mass value="0.072"/>
-        <inertia ixx="3.88e-6" ixy="0" ixz="0" iyy="4.99e-7" iyz="0" izz="3.88e-6"/>
-      </inertial>
+      <inertial><mass value="0.001"/><inertia ixx="1e-9" ixy="0" ixz="0" iyy="1e-9" iyz="0" izz="1e-9"/></inertial>
     </link>
-    <!-- ══════════════════════════════════════════════════════════════
-         FISHEYE CAMERA (广角单目, FOV diagonal 200°) — WN-L712V11
-         Posición sobre gripper_base: X=-73.5 mm (a lo largo del gripper),
-         Z=37 mm (altura). Y=0.
-         Malla: fisheye.stl (Ø22.65 × 20.2 mm, exportada de SolidWorks→Onshape)
-    ══════════════════════════════════════════════════════════════════ -->
     <joint name="${prefix}pika_fisheye_joint" type="fixed">
       <parent link="${prefix}gripper_base"/>
       <child  link="${prefix}pika_fisheye_link"/>
-      <origin xyz="-0.0735 0 0.037" rpy="-1.5708 0 0"/>
+      <origin xyz="-0.0799 0 0.0683" rpy="0 0 0"/>
     </joint>
     <link name="${prefix}pika_fisheye_link">
-      <visual>
-        <origin xyz="0 0 0" rpy="1.5708 0 0"/>
-        <geometry>
-          <mesh filename="package://pika_description/meshes/fisheye.stl"
-                scale="0.001 0.001 0.001"/>
-        </geometry>
-        <material name="${prefix}pika_dark"/>
-      </visual>
-      <collision>
-        <origin xyz="0 0 0.0045" rpy="1.5708 0 0"/>
-        <geometry><cylinder radius="0.0113" length="0.0202"/></geometry>
-      </collision>
-      <inertial>
-        <mass value="0.008"/>
-        <inertia ixx="1e-6" ixy="0" ixz="0" iyy="1e-6" iyz="0" izz="1e-6"/>
-      </inertial>
+      <inertial><mass value="0.001"/><inertia ixx="1e-9" ixy="0" ixz="0" iyy="1e-9" iyz="0" izz="1e-9"/></inertial>
     </link>
-    <!-- ══════════════════════════════════════════════════════════════
-         GARRAS — idéntico a joint7/joint8 + link7/link8 del Piper
-    ══════════════════════════════════════════════════════════════════ -->
-    <!-- Garra izquierda (link7) — idéntico a joint7 del Piper -->
-    <joint name="${prefix}pika_jaw_left_joint" type="prismatic">
-      <parent link="${prefix}gripper_base"/>
-      <child  link="${prefix}pika_jaw_left"/>
-      <origin xyz="0 0 0.1358" rpy="1.5708 0 0"/>
-      <axis xyz="0 0 1"/>
-      <limit lower="0" upper="0.035" effort="10.0" velocity="1.0"/>
-    </joint>
-    <link name="${prefix}pika_jaw_left">
-      <visual>
-        <origin xyz="0 0 0" rpy="0 0 0"/>
-        <geometry>
-          <mesh filename="package://pika_description/meshes/link7.STL"/>
-        </geometry>
-        <material name="${prefix}pika_dark"/>
-      </visual>
-      <collision>
-        <origin xyz="0 0 0" rpy="0 0 0"/>
-        <geometry>
-          <mesh filename="package://pika_description/meshes/link7.STL"/>
-        </geometry>
-      </collision>
-      <inertial>
-        <mass value="0.025"/>
-        <inertia ixx="7.4e-5" ixy="-1.1e-6" ixz="2.1e-7" iyy="-1.1e-6" iyz="-1.4e-5" izz="7.5e-5"/>
-      </inertial>
-    </link>
-    <!-- Garra derecha (link8) — idéntico a joint8 del Piper, sin mimic -->
-    <joint name="${prefix}pika_jaw_right_joint" type="prismatic">
-      <parent link="${prefix}gripper_base"/>
-      <child  link="${prefix}pika_jaw_right"/>
-      <origin xyz="0 0 0.1358" rpy="1.5708 0 -3.1416"/>
-      <axis xyz="0 0 -1"/>
-      <limit lower="-0.035" upper="0" effort="10.0" velocity="1.0"/>
-    </joint>
-    <link name="${prefix}pika_jaw_right">
-      <visual>
-        <origin xyz="0 0 0" rpy="0 0 0"/>
-        <geometry>
-          <mesh filename="package://pika_description/meshes/link8.STL"/>
-        </geometry>
-        <material name="${prefix}pika_dark"/>
-      </visual>
-      <collision>
-        <origin xyz="0 0 0" rpy="0 0 0"/>
-        <geometry>
-          <mesh filename="package://pika_description/meshes/link8.STL"/>
-        </geometry>
-      </collision>
-      <inertial>
-        <mass value="0.025"/>
-        <inertia ixx="7.4e-5" ixy="-1.1e-6" ixz="2.1e-7" iyy="-1.1e-6" iyz="-1.4e-5" izz="7.5e-5"/>
-      </inertial>
-    </link>
-    <!-- ── TCP (Tool Center Point) ──────────────────────────────────── -->
     <joint name="${prefix}pika_tcp_joint" type="fixed">
       <parent link="${prefix}gripper_base"/>
       <child  link="${prefix}pika_tcp"/>
-      <origin xyz="0 0 0.185" rpy="0 0 0"/>
+      <origin xyz="-0.00642 0 0.180" rpy="0 0 0"/>
     </joint>
     <link name="${prefix}pika_tcp"/>

File: src/pika_sim/urdf/pika_piper_gazebo.urdf.xacro (robot description, xacro)
@@ -44,8 +44,6 @@
   <xacro:color_gazebo link="link6" material="Gazebo/FlatBlack"/>
   <xacro:color_gazebo link="gripper_base" material="Gazebo/FlatBlack"/>
-  <xacro:color_gazebo link="pika_jaw_left" material="Gazebo/FlatBlack"/>
-  <xacro:color_gazebo link="pika_jaw_right" material="Gazebo/FlatBlack"/>
-  <xacro:color_gazebo link="pika_depth_link" material="Gazebo/Grey"/>
-  <xacro:color_gazebo link="pika_fisheye_link" material="Gazebo/Grey"/>
+  <xacro:color_gazebo link="pika_jaw_left" material="Gazebo/Grey"/>
+  <xacro:color_gazebo link="pika_jaw_right" material="Gazebo/Grey"/>
   <!-- ══════════════════════════════════════════════════════════════
        Cámaras simuladas del gripper Pika, con los topics del hardware real
@@ -57,6 +55,5 @@
          /gripper/camera/depth/color/points               D405 nube de puntos
          /gripper/camera_fisheye/color/image_raw          fisheye
-       Supuesto (igual que escena_nbv_demo.py): ambas miran a lo largo de +Z de gripper_base,
-       el eje de la herramienta. Las cámaras de Gazebo miran por +X de su link; de ahí el
+       Ambas miran a lo largo de +Z de gripper_base, el eje de la herramienta (plano de AgileX). Las cámaras de Gazebo miran por +X de su link; de ahí el
        giro (0, -π/2, 0). Los marcos ópticos siguen la convención de ROS (Z adelante, X a la
        derecha, Y abajo). Con camaras:=false no se cargan (Gazebo más liviano, p. ej. modo MIT).
@@ -65,7 +62,7 @@
   <xacro:if value="$(arg camaras)">
     <xacro:property name="PI" value="3.141592653589793"/>
-    <xacro:macro name="marco_camara" params="nombre xyz">
+    <xacro:macro name="marco_camara" params="nombre padre xyz">
       <joint name="${nombre}_joint" type="fixed">
-        <parent link="gripper_base"/>
+        <parent link="${padre}"/>
         <child link="${nombre}_link"/>
         <origin xyz="${xyz}" rpy="0 ${-PI/2} 0"/>
@@ -85,8 +82,9 @@
       <link name="${nombre}_optical_frame"/>
     </xacro:macro>
-    <!-- D405: frente del módulo, 12 mm por delante del centro de pika_depth_link -->
-    <xacro:marco_camara nombre="pika_d405" xyz="-0.046 0 0.039"/>
-    <!-- Fisheye: frente del lente, sobre pika_fisheye_link -->
-    <xacro:marco_camara nombre="pika_fisheye_cam" xyz="-0.0735 0 0.047"/>
+    <!-- Posiciones del modelo de AgileX (pika_description). La D405 real tiene el centro óptico 4 mm
+         detrás de la tapa, que en la malla es sólida: el sensor de Gazebo va 4 mm adelante para
+         dibujar desde fuera de la carcasa. -->
+    <xacro:marco_camara nombre="pika_d405" padre="pika_depth_link" xyz="0 0 0.004"/>
+    <xacro:marco_camara nombre="pika_fisheye_cam" padre="pika_fisheye_link" xyz="0 0 0.001"/>
     <!-- D405: 87° × 58°, 7–50 cm de rango útil; 640×480 a 30 Hz como start_single_gripper.bash -->
     <gazebo reference="pika_d405_link">
