Commit message: pika_sim: escena de demostracion de NBV con capturas de Gazebo
escena_nbv_demo.py:
- arma una escena con rama, fruta y hojas que la ocluyen
- genera 20 vistas en un casquete de 0.22 m y calcula para cada una la
  visibilidad (trazado de rayos contra las hojas) y si es alcanzable (IK
  de la D405 sobre el URDF, error < 5 mm y < 3 grados, |J5| > 10 grados)
- lleva el Piper a la mejor vista y captura con camaras virtuales la
  escena, la vista frontal y la elegida
panel_nbv.py arma la figura con los numeros del JSON.

Resultado: 7/20 vistas alcanzables (el limite de +-70 grados de J5 descarta
las laterales, altas y las que miran hacia arriba); la vista frontal ve el
0 % de la fruta y la mejor alcanzable el 50 %.

Colores AgileX del brazo en Gazebo (urdf/pika_piper_gazebo.urdf.xacro).
Figura y resultados en docs/percepcion_activa/lazos_cinematica_nbv.md (5.6).

Co-Authored-By: Claude Opus 5.5 <noreply@anthropic.com>

File: src/pika_sim/urdf/pika_piper_gazebo.urdf.xacro (robot description, xacro)
@@ -31,4 +31,21 @@
     <xacro:position_joint name="pika_jaw_right_joint"/>
   </ros2_control>
+  <!-- Colores AgileX en Gazebo (Gazebo Classic no usa los materiales del URDF): base y
+       articulaciones negras, brazo y antebrazo grafito, gripper Pika negro mate, cámaras plata -->
+  <xacro:macro name="color_gazebo" params="link material">
+    <gazebo reference="${link}"><material>${material}</material></gazebo>
+  </xacro:macro>
+  <xacro:color_gazebo link="base_link" material="Gazebo/FlatBlack"/>
+  <xacro:color_gazebo link="link1" material="Gazebo/FlatBlack"/>
+  <xacro:color_gazebo link="link2" material="Gazebo/DarkGrey"/>
+  <xacro:color_gazebo link="link3" material="Gazebo/DarkGrey"/>
+  <xacro:color_gazebo link="link4" material="Gazebo/FlatBlack"/>
+  <xacro:color_gazebo link="link5" material="Gazebo/FlatBlack"/>
+  <xacro:color_gazebo link="link6" material="Gazebo/FlatBlack"/>
+  <xacro:color_gazebo link="gripper_base" material="Gazebo/FlatBlack"/>
+  <xacro:color_gazebo link="pika_jaw_left" material="Gazebo/FlatBlack"/>
+  <xacro:color_gazebo link="pika_jaw_right" material="Gazebo/FlatBlack"/>
+  <xacro:color_gazebo link="pika_depth_link" material="Gazebo/Grey"/>
+  <xacro:color_gazebo link="pika_fisheye_link" material="Gazebo/Grey"/>
   <gazebo>
     <plugin filename="libgazebo_ros2_control.so" name="gazebo_ros2_control">

Commit message: Escenario de manzano y camaras simuladas del gripper Pika en pika_sim
- D405 (color, profundidad, nube) y fisheye en el gripper, con los topics
  /gripper/camera/... del hardware a 30 Hz; profundidad_mm.py publica la
  profundidad en 16UC1 mm como el driver real (data_tools convierte sin
  reescalar). Argumento camaras:=false para Gazebo liviano.
- escena_manzano.py: manzano reproducible por semilla, spawn en Gazebo y
  verdad del terreno en /escena/verdad (JSON) y /escena/frutas (MarkerArray).
  Launch: escena:=manzano semilla:=N.
- escena_nbv_demo.py usa el modulo y el arbol lanzado, y guarda lo que ven
  la D405 y la fisheye del gripper en la mejor vista.
- RViz: nube de la D405, manzanas e imagenes de ambas camaras.
- Documentacion: README de pika_sim, estado y contrato de percepcion activa,
  ejemplo del manzano con las imagenes de las camaras y AGENTS.md.

Co-Authored-By: Claude Opus 5.5 <noreply@anthropic.com>

File: src/pika_sim/urdf/pika_piper_gazebo.urdf.xacro (robot description, xacro)
@@ -48,4 +48,100 @@
   <xacro:color_gazebo link="pika_depth_link" material="Gazebo/Grey"/>
   <xacro:color_gazebo link="pika_fisheye_link" material="Gazebo/Grey"/>
+  <!-- ══════════════════════════════════════════════════════════════
+       Cámaras simuladas del gripper Pika, con los topics del hardware real
+       (config/single_pika_teleop_data_params.yaml de data_tools):
+         /gripper/camera/color/image_raw                  D405 color
+         /gripper/camera/aligned_depth_to_color/image_raw D405 profundidad, 16UC1 en mm como el
+                                                          driver real (profundidad_mm.py convierte
+                                                          los 32FC1 en metros de Gazebo)
+         /gripper/camera/depth/color/points               D405 nube de puntos
+         /gripper/camera_fisheye/color/image_raw          fisheye
+       Supuesto (igual que escena_nbv_demo.py): ambas miran a lo largo de +Z de gripper_base,
+       el eje de la herramienta. Las cámaras de Gazebo miran por +X de su link; de ahí el
+       giro (0, -π/2, 0). Los marcos ópticos siguen la convención de ROS (Z adelante, X a la
+       derecha, Y abajo). Con camaras:=false no se cargan (Gazebo más liviano, p. ej. modo MIT).
+  ══════════════════════════════════════════════════════════════════ -->
+  <xacro:arg name="camaras" default="true"/>
+  <xacro:if value="$(arg camaras)">
+    <xacro:property name="PI" value="3.141592653589793"/>
+    <xacro:macro name="marco_camara" params="nombre xyz">
+      <joint name="${nombre}_joint" type="fixed">
+        <parent link="gripper_base"/>
+        <child link="${nombre}_link"/>
+        <origin xyz="${xyz}" rpy="0 ${-PI/2} 0"/>
+      </joint>
+      <!-- inercia mínima: Gazebo descarta los links sin masa y con ellos el sensor -->
+      <link name="${nombre}_link">
+        <inertial>
+          <mass value="0.001"/>
+          <inertia ixx="1e-9" ixy="0" ixz="0" iyy="1e-9" iyz="0" izz="1e-9"/>
+        </inertial>
+      </link>
+      <joint name="${nombre}_optical_joint" type="fixed">
+        <parent link="${nombre}_link"/>
+        <child link="${nombre}_optical_frame"/>
+        <origin xyz="0 0 0" rpy="${-PI/2} 0 ${-PI/2}"/>
+      </joint>
+      <link name="${nombre}_optical_frame"/>
+    </xacro:macro>
+    <!-- D405: frente del módulo, 12 mm por delante del centro de pika_depth_link -->
+    <xacro:marco_camara nombre="pika_d405" xyz="-0.046 0 0.039"/>
+    <!-- Fisheye: frente del lente, sobre pika_fisheye_link -->
+    <xacro:marco_camara nombre="pika_fisheye_cam" xyz="-0.0735 0 0.047"/>
+    <!-- D405: 87° × 58°, 7–50 cm de rango útil; 640×480 a 30 Hz como start_single_gripper.bash -->
+    <gazebo reference="pika_d405_link">
+      <sensor type="depth" name="pika_d405">
+        <always_on>true</always_on>
+        <update_rate>30</update_rate>
+        <camera>
+          <horizontal_fov>1.518</horizontal_fov>
+          <image><width>640</width><height>480</height><format>R8G8B8</format></image>
+          <clip><near>0.02</near><far>1.5</far></clip>
+          <noise><type>gaussian</type><mean>0.0</mean><stddev>0.003</stddev></noise>
+        </camera>
+        <plugin name="pika_d405_driver" filename="libgazebo_ros_camera.so">
+          <ros>
+            <namespace>gripper</namespace>
+            <remapping>camera/image_raw:=camera/color/image_raw</remapping>
+            <remapping>camera/camera_info:=camera/color/camera_info</remapping>
+            <remapping>camera/depth/image_raw:=camera/depth_sim/image_raw</remapping>
+            <remapping>camera/depth/camera_info:=camera/aligned_depth_to_color/camera_info</remapping>
+            <remapping>camera/points:=camera/depth/color/points</remapping>
+          </ros>
+          <camera_name>camera</camera_name>
+          <frame_name>pika_d405_optical_frame</frame_name>
+          <min_depth>0.07</min_depth>
+          <max_depth>0.5</max_depth>
+        </plugin>
+      </sensor>
+    </gazebo>
+    <!-- Fisheye WN-L712V11 (200° en diagonal): lente equidistante de Gazebo, 180° en horizontal -->
+    <gazebo reference="pika_fisheye_cam_link">
+      <sensor type="wideanglecamera" name="pika_fisheye">
+        <always_on>true</always_on>
+        <update_rate>30</update_rate>
+        <camera>
+          <horizontal_fov>3.1416</horizontal_fov>
+          <image><width>640</width><height>480</height><format>R8G8B8</format></image>
+          <clip><near>0.01</near><far>20</far></clip>
+          <lens>
+            <type>equidistant</type>
+            <scale_to_hfov>true</scale_to_hfov>
+            <cutoff_angle>1.75</cutoff_angle>
+            <env_texture_size>512</env_texture_size>
+          </lens>
+        </camera>
+        <plugin name="pika_fisheye_driver" filename="libgazebo_ros_camera.so">
+          <ros>
+            <namespace>gripper</namespace>
+            <remapping>camera_fisheye/image_raw:=camera_fisheye/color/image_raw</remapping>
+            <remapping>camera_fisheye/camera_info:=camera_fisheye/color/camera_info</remapping>
+          </ros>
+          <camera_name>camera_fisheye</camera_name>
+          <frame_name>pika_fisheye_cam_optical_frame</frame_name>
+        </plugin>
+      </sensor>
+    </gazebo>
+  </xacro:if>
   <gazebo>
     <plugin filename="libgazebo_ros2_control.so" name="gazebo_ros2_control">
